Commit message: build test

File: rbim_description/urdf/ball.xacro (robot description, xacro)
@@ -28,4 +28,44 @@
 	    </collision>
 	</link>
+    <!--
+    Center of buoyancy according to eq. (3.1) p. 28 in Berg2012.
+    The original values, [0.0822, -0.00773, 0.3872] however, seem to
+    assume NWU (otherwise cob is below cog?).
+    -->
+    <xacro:property name="cob" value="0.0 0.0 0.3"/>
+    <!-- Volume, see p.31 in Berg2012 -->
+    <xacro:property name="volume" value="1.83826"/>
+    <xacro:macro name="ball_hydro_model">
+        <link name="ball/base_link">
+            <neutrally_buoyant>0</neutrally_buoyant>
+            <volume>${volume}</volume>
+            <box>
+                <width>1.5</width>
+                <length>2.6</length>
+                <height>1.6</height>
+            </box>
+            <center_of_buoyancy>${cob}</center_of_buoyancy>
+            <hydrodynamic_model>
+                <type>fossen</type>
+                <!-- Added mass: see p.28 in Berg2012 -->
+                <added_mass>
+                     779.79 -6.8773 -103.32  8.5426 -165.54 -7.8033
+                    -6.8773    1222   51.29  409.44 -5.8488  62.726
+                    -103.32   51.29  3659.9  6.1112 -386.42  10.774
+                     8.5426  409.44  6.1112   534.9 -10.027  21.019
+                    -165.54 -5.8488 -386.42 -10.027  842.69 -1.1162
+                    -7.8033  62.726  10.775  21.019 -1.1162  224.32
+                </added_mass>
+                <!-- Linear damping: see p.31 in Berg2012 -->
+                <linear_damping>
+                    -74.82 -69.48 -728.4 -268.8 -309.77 -105
+                </linear_damping>
+                <!-- Non-linear damping: see p.30 in Berg2012 -->
+                <quadratic_damping>
+                    -748.22 -992.53 -1821.01 -672 -774.44 -523.27
+                </quadratic_damping>
+            </hydrodynamic_model>
+        </link>
+    </xacro:macro>
     <gazebo reference="ball/base_link">
         <material>Gazebo/Blue</material>
@@ -36,7 +76,7 @@
         <fluid_density>1028.0</fluid_density>
         <flow_velocity_topic>hydrodynamics/current_velocity</flow_velocity_topic>
-        <!-- <debug>$(arg debug)</debug> -->
+        <debug>true</debug>
         <!-- Adding the hydrodynamic and hydrostatic parameters for the vehicle-->
-        <xacro:rexrov_hydro_model namespace="$(arg namespace)"/>
+        <xacro:ball_hydro_model />
       </plugin>
     </gazebo>

File: uuv_descriptions/urdf/rexrov_base.xacro (robot description, xacro)
@@ -26,5 +26,5 @@
   <xacro:include filename="$(find uuv_sensor_ros_plugins)/urdf/sensor_snippets.xacro"/>
 -->
-  <xacro:include filename="$(find uuv_gazebo_ros_plugins)/urdf/snippets.xacro"/>
+  <xacro:include filename="$(find uuv_gazebo_plugins)/urdf/snippets.xacro"/>
   <!-- Parameters -->
   <xacro:property name="namespace" value="rexrov"/>
@@ -71,14 +71,55 @@
       </collision>
     </link>
-    <!-- Set up hydrodynamic plugin given as input parameter -->
+    <!--
+    Center of buoyancy according to eq. (3.1) p. 28 in Berg2012.
+    The original values, [0.0822, -0.00773, 0.3872] however, seem to
+    assume NWU (otherwise cob is below cog?).
+    -->
+    <xacro:property name="cob" value="0.0 0.0 0.3"/>
+    <!-- Volume, see p.31 in Berg2012 -->
+    <xacro:property name="volume" value="1.83826"/>
+    <xacro:macro name="rexrov_hydro_model" params="namespace">
+        <link name="${namespace}/base_link">
+            <neutrally_buoyant>0</neutrally_buoyant>
+            <volume>${volume}</volume>
+            <box>
+                <width>1.5</width>
+                <length>2.6</length>
+                <height>1.6</height>
+            </box>
+            <center_of_buoyancy>${cob}</center_of_buoyancy>
+            <hydrodynamic_model>
+                <type>fossen</type>
+                <!-- Added mass: see p.28 in Berg2012 -->
+                <added_mass>
+                     779.79 -6.8773 -103.32  8.5426 -165.54 -7.8033
+                    -6.8773    1222   51.29  409.44 -5.8488  62.726
+                    -103.32   51.29  3659.9  6.1112 -386.42  10.774
+                     8.5426  409.44  6.1112   534.9 -10.027  21.019
+                    -165.54 -5.8488 -386.42 -10.027  842.69 -1.1162
+                    -7.8033  62.726  10.775  21.019 -1.1162  224.32
+                </added_mass>
+                <!-- Linear damping: see p.31 in Berg2012 -->
+                <linear_damping>
+                    -74.82 -69.48 -728.4 -268.8 -309.77 -105
+                </linear_damping>
+                <!-- Non-linear damping: see p.30 in Berg2012 -->
+                <quadratic_damping>
+                    -748.22 -992.53 -1821.01 -672 -774.44 -523.27
+                </quadratic_damping>
+            </hydrodynamic_model>
+        </link>
+    </xacro:macro>
 <!--
-    <xacro:insert_block name="gazebo"/>
+    <gazebo>
+      <plugin name="uuv_plugin" filename="libuuv_underwater_object_ros_plugin.so">
+        <fluid_density>1028.0</fluid_density>
+        <flow_velocity_topic>hydrodynamics/current_velocity</flow_velocity_topic>
+        <debug>$(arg debug)</debug>
+        Adding the hydrodynamic and hydrostatic parameters for the vehicle
+        <xacro:rexrov_hydro_model namespace="$(arg namespace)"/>
+      </plugin>
+    </gazebo>
 -->
-    <!-- optional: plugin to test compare Gazebo's returned accelerations
-    <gazebo>
-      <plugin name="${namespace}_test_plugin" filename="libuuv_accelerations_test_plugin.so">
-        <link_name>${namespace}/base_link</link_name>
-      </plugin>
-    </gazebo> -->
     <xacro:include filename="$(find uuv_descriptions)/urdf/rexrov_actuators.xacro"/>
 <!--
@@ -86,3 +127,5 @@
   </xacro:macro>
 -->
+  <!-- Joint state publisher plugin -->
+  <xacro:default_joint_state_publisher namespace="rexrov" update_rate="50"/>
 </robot>
