Commit message: remove unused files

File: uuv_control/uuv_thruster_manager/urdf/robot.urdf (robot description, URDF)
Before this commit: robot rexrov, 9 links, 8 joints
Links:
- link rexrov/base_link: geometry collision box size=2.20 0.10 1.10; collision box size=2.20 0.10 1.10
- link rexrov/thruster_0: geometry collision cylinder length=0.000001 radius=0.000001; visual mesh filename=file:///uuv_descriptions/meshes/prop.dae scale=1 1 1
- link rexrov/thruster_1: geometry collision cylinder length=0.000001 radius=0.000001; visual mesh filename=file:///uuv_descriptions/meshes/prop.dae scale=1 1 1
- link rexrov/thruster_2: geometry collision cylinder length=0.000001 radius=0.000001; visual mesh filename=file:///uuv_descriptions/meshes/prop.dae scale=1 1 1
- link rexrov/thruster_3: geometry collision cylinder length=0.000001 radius=0.000001; visual mesh filename=file:///uuv_descriptions/meshes/prop.dae scale=1 1 1
- link rexrov/thruster_4: geometry collision cylinder length=0.000001 radius=0.000001; visual mesh filename=file:///uuv_descriptions/meshes/prop.dae scale=1 1 1
- link rexrov/thruster_5: geometry collision cylinder length=0.000001 radius=0.000001; visual mesh filename=file:///uuv_descriptions/meshes/prop.dae scale=1 1 1
- link rexrov/thruster_6: geometry collision cylinder length=0.000001 radius=0.000001; visual mesh filename=file:///uuv_descriptions/meshes/prop.dae scale=1 1 1
- link rexrov/thruster_7: geometry collision cylinder length=0.000001 radius=0.000001; visual mesh filename=file:///uuv_descriptions/meshes/prop.dae scale=1 1 1
